Commit message: Prof

File: urdf/iiwa_7.urdf (robot description, URDF)
Before this commit: robot KUKA_iiwa, 9 links, 8 joints
Links:
- link link_0: geometry collision mesh filename=collision/link_0.stl; visual mesh filename=visual/link_0.glb
- link link_1: geometry collision mesh filename=collision/link_1.stl; visual mesh filename=visual/link_1.glb
- link link_2: geometry collision mesh filename=collision/link_2.stl; visual mesh filename=visual/link_2.glb
- link link_3: geometry collision mesh filename=collision/link_3.stl; visual mesh filename=visual/link_3.glb
- link link_4: geometry collision mesh filename=collision/link_4.stl; visual mesh filename=visual/link_4.glb
- link link_5: geometry collision mesh filename=collision/link_5.stl; visual mesh filename=visual/link_5.glb
- link link_6: geometry collision mesh filename=collision/link_6.stl; visual mesh filename=visual/link_6.glb
- link link_7: geometry collision mesh filename=collision/link_7.stl; visual mesh filename=visual/link_7.glb
Joints:
- joint joint_1: limit lower=-2.9670597283903604 upper=2.9670597283903604 effort=50 velocity=100 -> lower=-2.9670597283903604 upper=2.9670597283903604 effort=300 velocity=10
- joint joint_2: limit lower=-2.0943951023931953 upper=2.0943951023931953 effort=50 velocity=100 -> lower=-2.0943951023931953 upper=2.0943951023931953 effort=300 velocity=10; origin xyz=0 0 0.19 rpy=1.5707963267948966   0 3.141592653589793 -> xyz=0 0 0.19 rpy=1.5707963267948966 0 3.141592653589793
- joint joint_3: limit lower=-2.9670597283903604 upper=2.9670597283903604 effort=50 velocity=100 -> lower=-2.9670597283903604 upper=2.9670597283903604 effort=300 velocity=10
- joint joint_4: limit lower=-2.0943951023931953 upper=2.0943951023931953 effort=50 velocity=100 -> lower=-2.0943951023931953 upper=2.0943951023931953 effort=300 velocity=10
- joint joint_5: limit lower=-2.9670597283903604 upper=2.9670597283903604 effort=50 velocity=100 -> lower=-2.9670597283903604 upper=2.9670597283903604 effort=300 velocity=10
- joint joint_6: limit lower=-2.0943951023931953 upper=2.0943951023931953 effort=50 velocity=100 -> lower=-2.0943951023931953 upper=2.0943951023931953 effort=300 velocity=10
- joint joint_7: limit lower=-3.0543261909900767 upper=3.0543261909900767 effort=50 velocity=100 -> lower=-3.0543261909900767 upper=3.0543261909900767 effort=300 velocity=10
